File: bldc_servo_mini_v1.kicad_sch (KiCad schematic)
At the start: 57 parts, among them IC1 DRV8313PWP, J1 Conn_01x05_MountingPin, J3 Conn_01x03, J6 Conn_01x05_MountingPin, U3 SN65HVD234, U5 STM32G431CBUx

Commit message: wip
Parts:
- removed U1, U4: ~, SC60228:SOIC-8_L5.0-W4.0-P1.27-LS6.0-BL, symbol SC60228:SC60228DC
- added U1, U2: MT6701QT, Package_DFN_QFN:QFN-16-1EP_3x3mm_P0.5mm_EP1.7x1.7mm, symbol Sensor_Magnetic:MT6701QT
Connections:
- net +3.3V: now also U2.13 (VDD), U2.14 (MODE)
- net CAN_EN: now also U5.47 (PB9); no longer U5.12 (PA4)
- net CS: now also U2.8 (Z); no longer FPC_BOARD1.6
- net GND: now also U2.16 (GND), U2.17 (GND)
- net MISO: now also U2.6 (A)
- net SCK: now also U2.7 (B)
- net SENSOR2_3V3: now also U1.13 (VDD), U1.14 (MODE)
- net SENSOR2_CS: now also U1.8 (Z)
- net SENSOR2_GND: now also U1.16 (GND), U1.17 (GND)
- net SENSOR2_MISO: now also U1.6 (A)
- net SENSOR2_SCK: now also U1.7 (B)
- new net CS_EXTERNAL: FPC_BOARD1.6, U5.12 (PA4)
- no-connect marks 10 -> 16
Other:
- moved on the sheet: C11, C7

Commit message: 6 layer board draft
Parts:
- removed C12, C8: 10u, Capacitor_SMD:C_0805_2012Metric_Pad1.18x1.45mm_HandSolder, symbol Device:C_Small
- removed C14, C15, C30, C32: 100n, Capacitor_SMD:C_0402_1005Metric_Pad0.74x0.62mm_HandSolder, symbol Device:C_Small
- removed H2: MountingHole_Pad, MountingHole:MountingHole_2.2mm_M2_Pad_TopBottom, symbol Mechanical:MountingHole_Pad
- removed IC1: DRV8313PWP, DRV8313PWP:SOP65P640X120-29N, symbol DRV8313PWP:DRV8313PWP
- removed J3: Conn_01x03, Connector_JST:JST_PH_S3B-PH-SM4-TB_1x03-1MP_P2.00mm_Horizontal, symbol Connector_Generic:Conn_01x03
- removed J5: ~, positive_altitude:Positive_Altitude_SWD_Connector_V2, symbol positive_altitude:Positive_Altitude_SWD_Connector_V2
- removed NT1, NT2, NT3: NetTie_2, positive_altitude:NetTie-2_SMD_Pad0.2mm, symbol Device:NetTie_2
- removed R13, R16, R29: 10m, 0.1W+, 0603, Resistor_SMD:R_0603_1608Metric_Pad0.98x0.95mm_HandSolder, symbol Device:R_Small
- removed R19, R21, R25: 67k, Resistor_SMD:R_0402_1005Metric_Pad0.72x0.64mm_HandSolder, symbol Device:R_Small
- removed R20, R22, R23, R24, R26, R27: 2.2k, Resistor_SMD:R_0402_1005Metric_Pad0.72x0.64mm_HandSolder, symbol Device:R_Small
- removed U3: SN65HVD234, Package_SO:SOIC-8_3.9x4.9mm_P1.27mm, symbol Interface_CAN_LIN:SN65HVD234
- removed U5: STM32G431CBUx, Package_DFN_QFN:QFN-48-1EP_7x7mm_P0.5mm_EP5.6x5.6mm, symbol MCU_ST_STM32G4:STM32G431CBUx
- added C17, C20: 100n, Capacitor_SMD:C_0402_1005Metric_Pad0.74x0.62mm_HandSolder, symbol Device:C_Small
- added C18: 22u, Capacitor_SMD:C_1210_3225Metric_Pad1.33x2.70mm_HandSolder, symbol Device:C_Small
- added C19: 100u, Capacitor_SMD:CP_Elec_6.3x5.8, symbol Device:C_Polarized_Small
- added IC2: DRV8311HRRWR, DRV8311HRRWR:DRV8311PRRWR, symbol DRV8311HRRWR:DRV8311HRRWR
- added J2: Positive_Altitude_SWD_Connector, positive_altitude:Positive_Altitude_SWD_Connector, symbol positive_altitude:Positive_Altitude_SWD_Connector
- added J4: Conn_01x03_MountingPin, Connector_JST:JST_PH_S3B-PH-SM4-TB_1x03-1MP_P2.00mm_Horizontal, symbol Connector_Generic_MountingPin:Conn_01x03_MountingPin
- added JP2: SolderJumper_2_Open, Jumper:SolderJumper-2_P1.3mm_Open_RoundedPad1.0x1.5mm, symbol Jumper:SolderJumper_2_Open
- added R1: 47k, Resistor_SMD:R_0402_1005Metric_Pad0.72x0.64mm_HandSolder, symbol Device:R_Small
- added U3: SN65HVD230, Package_SO:SOIC-8_3.9x4.9mm_P1.27mm, symbol Interface_CAN_LIN:SN65HVD230
- added U4: STM32G431KBUx, Package_DFN_QFN:QFN-32-1EP_5x5mm_P0.5mm_EP3.45x3.45mm, symbol MCU_ST_STM32G4:STM32G431KBUx
- C16: value 10n -> 4.7u; footprint Capacitor_SMD:C_0402_1005Metric_Pad0.74x0.62mm_HandSolder -> Capacitor_SMD:C_0603_1608Metric_Pad1.08x0.95mm_HandSolder
- C9: value 470n -> 100n
- D2: value TVS 26V -> TVS 17V
- PAD4: value VIN -> GND
- PAD5: value GND -> VCC
Connections:
- net +3.3V: now also J2.1 (+3.3V), JP2.2 (B), U3.3 (VCC), U4.1 (VDD), U4.17 (VDD)
- net CAN_H: now also R3.2, U3.7 (CANH); no longer JP1.1 (A)
- net CAN_L: now also JP1.1 (A), U3.6 (CANL); no longer R3.2
- net CAN_RX: now also U3.4 (R), U4.21 (PA11)
- net CAN_TX: now also U3.1 (D), U4.22 (PA12)
- net CS: now also U4.9 (PA4)
- net CS_EXTERNAL: now also U4.25 (PA15)
- net DRIVER_NFAULT: now also IC2.1 (NFAULT), U4.3 (PF1)
- net DRIVER_NSLEEP: now also IC2.24 (NSLEEP), U4.8 (PA3)
- net GND: now also C16.2, PAD4.1, C17.2, C18.2, C19.2, C20.2, IC2.16 (AGND), IC2.25 (EP), IC2.9 (PGND), J2.3 (GND), R1.2, U3.2 (GND), U3.8 (Rs), U4.14 (VSSA), U4.16 (VSS), U4.31 (PB8), U4.32 (VSS), U4.33 (VSS); no longer PAD5.1
- net MISO: now also U4.27 (PB4)
- net MOSI: now also U4.28 (PB5)
- net NRST: now also J2.5 (RESET), U4.4 (PG10)
- net OUT1: now also IC2.10 (OUTA), J4.1 (Pin_1)
- net OUT2: now also IC2.11 (OUTB), J4.2 (Pin_2)
- net OUT3: now also IC2.12 (OUTC), J4.3 (Pin_3)
- net SCK: now also U4.26 (PB3)
- net SWCLK: now also J2.2 (SWCLK), U4.24 (PA14)
- net SWDIO: now also J2.4 (SWDIO), U4.23 (PA13)
- net VCC: now also C6.1, C9.1, PAD5.1, C17.1, C18.1, C19.1, IC2.7 (VIN_AVDD), IC2.8 (VM); no longer C6.2, PAD4.1
- net VDDA: now also C20.1, IC2.2 (CSAREF), U4.15 (VDDA)
- net VOLTAGE_SENCE: now also U4.11 (PA6)
- net DRIVER_AVDD: now reaches C16.1
- net DRIVER_AVDD: now also IC2.17 (AVDD), JP2.1 (A)
- new net CURRENT1: IC2.5 (SOA), U4.7 (PA2)
- new net CURRENT2: IC2.4 (SOB), U4.6 (PA1)
- new net CURRENT3: IC2.3 (SOC), U4.5 (PA0)
- new net DRIVER_CP: C6.2, IC2.6 (CP)
- new net DRIVER_GAIN: IC2.21 (GAIN), U4.29 (PB6)
- new net DRIVER_MODE: IC2.23 (MODE), R1.1
- new net DRIVER_SLEW: IC2.22 (SLEW), U4.30 (PB7)
- new net PWM_H1: IC2.15 (INHA), U4.18 (PA8)
- new net PWM_H2: IC2.14 (INHB), U4.19 (PA9)
- new net PWM_H3: IC2.13 (INHC), U4.20 (PA10)
- new net PWM_L1: IC2.18 (INLA), U4.12 (PA7)
- new net PWM_L2: IC2.19 (INLB), U4.13 (PB0)
- new net PWM_L3: IC2.20 (INLC), U4.2 (PF0)
- no-connect marks 16 -> 19
Other:
- note added: "Cap: GYC1V470MCQ1GS"
- moved on the sheet: C1, C10, C13, C2, C3, C33, C4, C5, D2, FB1, JP1, PAD4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

Commit message: Component IDs and cleanup
Parts:
- removed C11: 100n, Capacitor_SMD:C_0402_1005Metric_Pad0.74x0.62mm_HandSolder, symbol Device:C_Small
- removed FPC_SENSOR2: FPC-8PIN, HCTL HC-FPC-05-09-8RLTAG:FPC-SMD_8P-P0.50_HC-FPC-05-09-8RLTAG, symbol HCTL HC-FPC-05-09-8RLTAG:HC-FPC-05-09-8RLTAG
- removed H5, H6: MountingHole_Pad, MountingHole:MountingHole_2.2mm_M2_Pad_TopBottom, symbol Mechanical:MountingHole_Pad
- removed U1: MT6701QT, Package_DFN_QFN:QFN-16-1EP_3x3mm_P0.5mm_EP1.7x1.7mm, symbol Sensor_Magnetic:MT6701QT
- C1, C16: LCSC (none) -> C162274
- C10, C13, C17, C2, C20, C3, C33, C6, C7, C9: LCSC (none) -> C77020
- C18: LCSC (none) -> C21397
- C19: value 100u -> 47u; LCSC (none) -> C2161781
- C4: value 1u -> 4.7u; LCSC (none) -> C162274
- C5: LCSC (none) -> C77019
- D2: LCSC (none) -> C353303
- FB1: LCSC (none) -> C710336
- FPC1: renamed from FPC_BOARD1; value FPC-8PIN -> External_sensor; LCSC (none) -> C5213749
- H1, J2, PAD4, PAD5: LCSC (none) -> -
- IC2: LCSC (none) -> C5218862
- J1: value Conn_01x05_MountingPin -> Power_and_data1; LCSC (none) -> C136657
- J4: value Conn_01x03_MountingPin -> Motor_connector; LCSC (none) -> C265101
- J6: value Conn_01x05_MountingPin -> Power_and_data2; LCSC (none) -> C136657
- JP1: value SolderJumper_2_Open -> Enable_CAN_termination; LCSC (none) -> -
- JP2: value SolderJumper_2_Open -> Enable_3.3V_source; LCSC (none) -> -
- R1: LCSC (none) -> C93943
- R3: LCSC (none) -> C114758
- R4: value 22k -> 47k; LCSC (none) -> C93943
- R5: value 4.7k -> 5.1k; LCSC (none) -> C105872
- U2: LCSC (none) -> C2913974
- U3: LCSC (none) -> C12084
- U4: LCSC (none) -> C1341901
Connections:
- net VOLTAGE_SENCE: now also U4.10 (PA5)
- no-connect marks 19 -> 11
Other:
- note added: "CAN Transciever 3.3V SN65HVD230"
- note added: "Connectors"
- note added: "Driver: 3 half bridges with low side current sensors DRV8311"
- note added: "MCU STM32G431KBU3"
- note added: "Magnetic Encoder: SPI, 14 bit MT6701"
- note added: "Solder Jumper: Enables 3.3V onboard source (provided from the driver)"
- note added: "Solder Jumper: Enables CAN bus termination resistor"
- note removed: "Cap: GYC1V470MCQ1GS"
- moved on the sheet: C1, C10, C13, C16, C17, C18, C19, C2, C20, C3, C33, C4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

Commit message: Upgrading to KiCad 9
Changed lines of the file:
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@@
 (kicad_sch
-	(version 20231120)
+	(version 20250114)
 	(generator "eeschema")
-	(generator_version "8.0")
+	(generator_version "9.0")
 	(paper "A4")
+	(text "MCU\nSTM32G431KBU3"
+		(exclude_from_sim no)
+		(at 15.494 18.288 0)
+		(effects
+			(font
+				(size 2 2)
+				(thickness 0.4)
+				(bold yes)
+			)
+			(justify left)
+		)
+	)
+	(text "Solder Jumper: Enables 3.3V\nonboard source \n(provided from the driver)"
+		(exclude_from_sim no)
+		(at 234.696 134.112 0)
+		(effects
+			(font
+				(size 2 2)
+				(thickness 0.4)
+				(bold yes)
+			)
+			(justify left)
+		)
+	)
+	(text "Driver: 3 half bridges with low side current sensors\nDRV8311"
+		(exclude_from_sim no)
+		(at 180.594 18.288 0)
+		(effects
+			(font
+				(size 2 2)
+				(thickness 0.4)
+				(bold yes)
+			)
+			(justify left)
+		)
+	)
+	(text "Magnetic Encoder: SPI, 14 bit\nMT6701"
+		(exclude_from_sim no)
+		(at 94.996 95.758 0)
+		(effects
+			(font
+				(size 2 2)
+				(thickness 0.4)
+				(bold yes)
+			)
+			(justify left)
+		)
+	)
+	(text "CAN Transciever 3.3V\nSN65HVD230"
+		(exclude_from_sim no)
+		(at 14.478 96.012 0)
+		(effects
+			(font
+				(size 2 2)
+				(thickness 0.4)
+				(bold yes)
+			)
+			(justify left)
+		)
+	)
+	(text "Solder Jumper: Enables CAN bus \ntermination resistor"
+		(exclude_from_sim no)
+		(at 179.324 132.588 0)
+		(effects
+			(font
+				(size 2 2)
+				(thickness 0.4)
+				(bold yes)
+			)
+			(justify left)
+		)
+	)
+	(text "Connectors"
+		(exclude_from_sim no)
+		(at 13.208 147.574 0)
+		(effects
+			(font
+				(size 2 2)
+				(thickness 0.4)
+				(bold yes)
+			)
+			(justify left)
+		)
+	)
 	(junction
 		(at 111.76 41.91)
@@
 		)
 	)
-	(text "MCU\nSTM32G431KBU3"
-		(exclude_from_sim no)
-		(at 15.494 18.288 0)
-		(effects
-			(font
-				(size 2 2)
-				(thickness 0.4)
-				(bold yes)
-			)
-			(justify left)
-		)
-	)
-	(text "Solder Jumper: Enables 3.3V\nonboard source \n(provided from the driver)"
-		(exclude_from_sim no)
-		(at 234.696 134.112 0)
-		(effects
-			(font
-				(size 2 2)
-				(thickness 0.4)
-				(bold yes)
-			)
-			(justify left)
-		)
-	)
-	(text "Driver: 3 half bridges with low side current sensors\nDRV8311"
-		(exclude_from_sim no)
-		(at 180.594 18.288 0)
-		(effects
-			(font
-				(size 2 2)
-				(thickness 0.4)
-				(bold yes)
-			)
-			(justify left)
-		)
-	)
-	(text "Magnetic Encoder: SPI, 14 bit\nMT6701"
-		(exclude_from_sim no)
-		(at 94.996 95.758 0)
-		(effects
-			(font
-				(size 2 2)
-				(thickness 0.4)
-				(bold yes)
-			)
-			(justify left)
-		)
-	)
-	(text "CAN Transciever 3.3V\nSN65HVD230"
-		(exclude_from_sim no)
-		(at 14.478 96.012 0)
-		(effects
-			(font
-				(size 2 2)
-				(thickness 0.4)
-				(bold yes)
-			)
-			(justify left)
-		)
-	)
-	(text "Solder Jumper: Enables CAN bus \ntermination resistor"
-		(exclude_from_sim no)
-		(at 179.324 132.588 0)
-		(effects
-			(font
-				(size 2 2)
-				(thickness 0.4)
-				(bold yes)
-			)
-			(justify left)
-		)
-	)
-	(text "Connectors"
-		(exclude_from_sim no)
-		(at 13.208 147.574 0)
-		(effects
-			(font
-				(size 2 2)
-				(thickness 0.4)
-				(bold yes)
-			)
-			(justify left)
-		)
-	)
 	(label "OUT1"
 		(at 247.65 86.36 270)
@@
 		)
 	)
+	(embedded_fonts no)
 )
