File: bldc_servo_v1.kicad_sch (KiCad schematic)
At the start: 36 parts, among them IC2 DRV8311HRRWR, J1 Power_and_data1, J2 Positive_Altitude_SWD_Connect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, J4 Motor_connector, J6 Power_and_data2, U2 MT6701QT, U3 SN65HVD230, U4 STM32G431KBUx

Commit message: Fabrication output
Parts:
- J2, PAD4, PAD5: now left out of the parts list
Changed lines of the file:
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@@
 		(at 36.83 186.69 0)
 		(unit 1)
-		(exclude_from_sim yes)
+		(exclude_from_sim no)
 		(in_bom no)
 		(on_board yes)
@@
 		(at 264.16 154.94 90)
 		(unit 1)
-		(exclude_from_sim yes)
+		(exclude_from_sim no)
 		(in_bom no)
 		(on_board yes)
@@
 		(unit 1)
 		(exclude_from_sim no)
-		(in_bom yes)
+		(in_bom no)
 		(on_board yes)
 		(dnp no)
@@
 		(unit 1)
 		(exclude_from_sim no)
-		(in_bom yes)
+		(in_bom no)
 		(on_board yes)
 		(dnp no)
@@
 		(at 212.09 154.94 90)
 		(unit 1)
-		(exclude_from_sim yes)
+		(exclude_from_sim no)
 		(in_bom no)
 		(on_board yes)
@@
 		(unit 1)
 		(exclude_from_sim no)
-		(in_bom yes)
+		(in_bom no)
 		(on_board yes)
 		(dnp no)
